File: hardware/controlboard/gp-controlboard/gp-controlboard.kicad_pcb (KiCad board)
At the start: 2 copper layers, 140 x 70 mm, 56 parts, among them J101 JUMPER-2_1, J102 JUMPER-2_1, J103 JUMPER-2_1, P101 BATTERY, P102 EN_JMP, P103 NUCLEO-CN3, P104 NUCLEO-CN4, P105 ESP_PROG, P106 BOOT_JMP, SW101 430162073826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

Commit message: Fixed silkscreen of control board
Parts:
- added G***: LOGO, EXTLOGO:GIAMMABOT_35MM_FSILK, F.Cu at (215.1, 90.5)
- added G***: LOGO, EXTLOGO:LOGO_OSH_15MM_FSILK, B.Cu at (206.2, 110.9)
- added G***: LOGO, EXTLOGO:LOGO_CC-BY-SA_20MM_FSILK, B.Cu at (139.9, 112.0)
- added VAL**: FIDUCIALMARK_1MM_3MM, MECHANICAL:FIDUCIALMARK_1MM_3MM, F.Cu at (155.0, 135.0)
- added VAL**: FIDUCIALMARK_1MM_3MM, MECHANICAL:FIDUCIALMARK_1MM_3MM, F.Cu at (235.0, 75.0)
- added VAL**: FIDUCIALMARK_1MM_3MM, MECHANICAL:FIDUCIALMARK_1MM_3MM, F.Cu at (105.0, 75.0)
Routing:
- net GND: vias 12 -> 20
Other:
- board text added: "by GIAMMATeam"
